File: CustomBoard/PowerSwitchClientBoard/PowerSwitchClientBoard.sch (KiCad schematic (older format))
At the start: 24 parts, among them J1 Conn_01x02, J2 Conn_01x02, J3 Conn_01x02, J4 Conn_01x02, J5 Conn_01x02, J6 Conn_01x02, J7 Conn_01x02, K1 G5LE-1, K2 G5LE-1, Q1 Q_NPN_EBC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

Commit message: WIP, got docker node/mqtt server working, can't get esphome devices to connect to it through mqtt.
Parts:
- removed D3, D4: LED, symbol PowerSwitchClientBoardLibrary:LED
Connections:
- no-connect marks 27 -> 23
Other:
- note added: "Also switch relays to thyristors"
- note added: "Need to replace PS with https://www.digikey.ca/product-detail/en/cui-inc/PBO-3-S9/102-4066-ND/6362755"
Changed lines of the file:
@@
 	2850 5000 3000 5000
-$Comp
-L PowerSwitchClientBoardLibrary:LED D3
-U 1 1 5D4ECCB4
-P 9250 2700
-F 0 "D3" V 9289 2583 50  0000 R CNN
-F 1 "LED" V 9198 2583 50  0000 R CNN
-F 2 "" H 9250 2700 50  0001 C CNN
-F 3 "https://www.lumex.com/content/files/ProductAttachment/SSI-LXH600GD-150.pdf" H 9250 2700 50  0001 C CNN
-F 4 "SSI-LXH600GD-150 " H 9250 2700 50  0001 C CNN "PartNumber"
-	1    9250 2700
-	0    -1   -1   0
-$EndComp
-$Comp
-L PowerSwitchClientBoardLibrary:LED D4
-U 1 1 5D4EF2EF
-P 9250 3450
-F 0 "D4" V 9289 3333 50  0000 R CNN
-F 1 "LED" V 9198 3333 50  0000 R CNN
-F 2 "" H 9250 3450 50  0001 C CNN
-F 3 "https://www.lumex.com/content/files/ProductAttachment/SSI-LXH600GD-150.pdf" H 9250 3450 50  0001 C CNN
-F 4 "SSI-LXH600GD-150 " H 9250 3450 50  0001 C CNN "PartNumber"
-	1    9250 3450
-	0    -1   -1   0
-$EndComp
 $Comp
 L PowerSwitchClientBoardLibrary:SW_Push SW1
@@
 	-1   0    0    1
 $EndComp
-NoConn ~ 9250 2550
-NoConn ~ 9250 2850
-NoConn ~ 9250 3300
-NoConn ~ 9250 3600
 $Comp
 L PowerSwitchClientBoardLibrary:R R4
@@
 Wire Wire Line
 	3000 1800 3050 1800
+Text Notes 3450 1050 0    50   ~ 0
+Need to replace PS with https://www.digikey.ca/product-detail/en/cui-inc/PBO-3-S9/102-4066-ND/6362755
+Text Notes 4550 1600 0    50   ~ 0
+Also switch relays to thyristors
 $EndSCHEMATC
